Commit message: chassis top box

File: description/robot_core.xacro (robot description, xacro)
@@ -66,4 +66,19 @@
         -->
     </link>
+    <!-- CHASSIS TOP -->
+    <joint name="chassis_top_joint" type="fixed">
+        <parent link="base_link"/>
+        <child link="chassis_top"/>
+        <origin xyz="${-wheel_offset_x} 0 ${chassis_height-wheel_offset_z}"/>
+    </joint>
+    <link name="chassis_top">
+        <visual>
+            <origin xyz="0.025 0 ${(chassis_height/2)-wheel_offset_z}"/>
+            <geometry>
+                <box size="0.05 ${chassis_width} ${chassis_height}"/>
+            </geometry>
+            <material name="white"/>
+        </visual>
+    </link>
     <!-- LEFT WHEEL LINK -->
     <joint name="left_wheel_joint" type="continuous">

Commit message: created caster wheel

File: description/robot_core.xacro (robot description, xacro)
@@ -11,5 +11,5 @@
     <xacro:property name="wheel_offset_y" value="0.048"/><!---->
     <xacro:property name="wheel_offset_z" value="0.005"/><!---->
-    <xacro:property name="caster_wheel_radius" value="0.01"/>
+    <xacro:property name="caster_wheel_radius" value="0.015"/>
     <xacro:property name="caster_wheel_mass" value="0.01"/>
     <xacro:property name="caster_wheel_offset_x" value="0.075"/>
@@ -137,3 +137,32 @@
     </gazebo>
     -->
+    <!-- CASTER WHEEL LINK -->
+    <joint name="caster_wheel_joint" type="fixed">
+        <parent link="chassis"/>
+        <child link="caster_wheel"/>
+        <origin xyz="${caster_wheel_offset_x} 0 ${caster_wheel_offset_z}"/>
+    </joint>
+    <link name="caster_wheel">
+        <visual>
+            <geometry>
+                <sphere radius="${caster_wheel_radius}"/>
+            </geometry>
+            <material name="white"/>
+        </visual>
+        <!--<collision>
+            <geometry>
+                <sphere radius="${caster_wheel_radius}"/>
+            </geometry>
+        </collision>
+        <xacro:inertial_sphere mass="${caster_wheel_mass}" radius="${caster_wheel_radius}">
+            <origin xyz="0 0 0" rpy="0 0 0"/>
+        </xacro:inertial_sphere>
+        -->
+    </link>
+    <!--<gazebo reference="caster_wheel">
+        <material>Gazebo/White</material>
+        <mu1 value="0.001"/>
+        <mu2 value="0.001"/>
+    </gazebo>
+    -->
 </robot>

Commit message: added inertia & collision

File: description/robot_core.xacro (robot description, xacro)
@@ -1,4 +1,5 @@
 <?xml version="1.0"?>
 <robot xmlns:xacro="http://www.ros.org/wiki/xacro"  >
+    <xacro:include filename="inertial_macros.xacro"/>
     <xacro:property name="chassis_length" value="0.09"/><!---->
     <xacro:property name="chassis_width" value="0.07"/><!---->
@@ -11,7 +12,7 @@
     <xacro:property name="wheel_offset_y" value="0.048"/><!---->
     <xacro:property name="wheel_offset_z" value="0.005"/><!---->
-    <xacro:property name="caster_wheel_radius" value="0.015"/>
+    <xacro:property name="caster_wheel_radius" value="0.015"/><!---->
     <xacro:property name="caster_wheel_mass" value="0.01"/>
-    <xacro:property name="caster_wheel_offset_x" value="0.075"/>
+    <xacro:property name="caster_wheel_offset_x" value="0.075"/><!---->
     <xacro:property name="caster_wheel_offset_z" value="${wheel_offset_z - wheel_radius + caster_wheel_radius}"/>
     <material name="white">
@@ -55,5 +56,5 @@
             <material name="white"/>
         </visual>
-        <!--<collision>
+        <collision>
             <origin xyz="${chassis_length/2} 0 ${chassis_height/2}"/>
             <geometry>
@@ -64,5 +65,4 @@
             <origin xyz="${chassis_length/2} 0 ${chassis_height/2}" rpy="0 0 0"/>
         </xacro:inertial_box>
-        -->
     </link>
     <!-- CHASSIS TOP -->
@@ -80,4 +80,13 @@
             <material name="white"/>
         </visual>
+        <collision>
+            <origin xyz="0.025 0 ${(chassis_height/2)-wheel_offset_z}"/>
+            <geometry>
+                <box size="0.05 ${chassis_width} ${chassis_height}"/>
+            </geometry>
+        </collision>
+        <xacro:inertial_box mass="0.5" x="${chassis_length}" y="${chassis_width}" z="${chassis_height}">
+            <origin xyz="0.025 0 ${(chassis_height/2)-wheel_offset_z}" rpy="0 0 0"/>
+        </xacro:inertial_box>
     </link>
     <!-- LEFT WHEEL LINK -->
@@ -95,5 +104,5 @@
             <material name="black"/>
         </visual>
-        <!--<collision>
+        <collision>
             <geometry>
                 <sphere radius="${wheel_radius}"/>
@@ -103,5 +112,4 @@
             <origin xyz="0 0 0" rpy="0 0 0"/>
         </xacro:inertial_cylinder>
-        -->
     </link>
     <!--<gazebo reference="left_wheel">
@@ -123,5 +131,5 @@
             <material name="black"/>
         </visual>
-        <!--<collision>
+        <collision>
             <geometry>
                 <sphere radius="${wheel_radius}"/>
@@ -131,5 +139,4 @@
             <origin xyz="0 0 0" rpy="0 0 0"/>
         </xacro:inertial_cylinder>
-        -->
     </link>
     <!--<gazebo reference="right_wheel">
@@ -150,5 +157,5 @@
             <material name="white"/>
         </visual>
-        <!--<collision>
+        <collision>
             <geometry>
                 <sphere radius="${caster_wheel_radius}"/>
@@ -158,5 +165,4 @@
             <origin xyz="0 0 0" rpy="0 0 0"/>
         </xacro:inertial_sphere>
-        -->
     </link>
     <!--<gazebo reference="caster_wheel">

Commit message: drive through GAZEBO

File: description/robot_core.xacro (robot description, xacro)
@@ -66,4 +66,7 @@
         </xacro:inertial_box>
     </link>
+    <gazebo reference="chassis">
+        <material>Gazebo/White</material>
+    </gazebo>
     <!-- CHASSIS TOP -->
     <joint name="chassis_top_joint" type="fixed">
@@ -86,8 +89,11 @@
             </geometry>
         </collision>
-        <xacro:inertial_box mass="0.5" x="${chassis_length}" y="${chassis_width}" z="${chassis_height}">
+        <xacro:inertial_box mass="0.03" x="${chassis_length}" y="${chassis_width}" z="${chassis_height}">
             <origin xyz="0.025 0 ${(chassis_height/2)-wheel_offset_z}" rpy="0 0 0"/>
         </xacro:inertial_box>
     </link>
+    <gazebo reference="chassis_top">
+        <material>Gazebo/White</material>
+    </gazebo>
     <!-- LEFT WHEEL LINK -->
     <joint name="left_wheel_joint" type="continuous">
@@ -113,8 +119,7 @@
         </xacro:inertial_cylinder>
     </link>
-    <!--<gazebo reference="left_wheel">
-        <material>Gazebo/Blue</material>
+    <gazebo reference="left_wheel">
+        <material>Gazebo/Black</material>
     </gazebo>
-    -->
     <!-- RIGHT WHEEL LINK -->
     <joint name="right_wheel_joint" type="continuous">
@@ -140,8 +145,7 @@
         </xacro:inertial_cylinder>
     </link>
-    <!--<gazebo reference="right_wheel">
-        <material>Gazebo/Blue</material>
+    <gazebo reference="right_wheel">
+        <material>Gazebo/Black</material>
     </gazebo>
-    -->
     <!-- CASTER WHEEL LINK -->
     <joint name="caster_wheel_joint" type="fixed">
@@ -166,9 +170,8 @@
         </xacro:inertial_sphere>
     </link>
-    <!--<gazebo reference="caster_wheel">
-        <material>Gazebo/White</material>
+    <gazebo reference="caster_wheel">
+        <material>Gazebo/Black</material>
         <mu1 value="0.001"/>
         <mu2 value="0.001"/>
     </gazebo>
-    -->
 </robot>

Commit message: mass correction

File: description/robot_core.xacro (robot description, xacro)
@@ -8,10 +8,10 @@
     <xacro:property name="wheel_radius" value="0.022"/><!---->
     <xacro:property name="wheel_thickness" value="0.017"/><!---->
-    <xacro:property name="wheel_mass" value="0.05"/>
+    <xacro:property name="wheel_mass" value="0.1"/>
     <xacro:property name="wheel_offset_x" value="0.016"/><!---->
     <xacro:property name="wheel_offset_y" value="0.048"/><!---->
     <xacro:property name="wheel_offset_z" value="0.005"/><!---->
     <xacro:property name="caster_wheel_radius" value="0.015"/><!---->
-    <xacro:property name="caster_wheel_mass" value="0.01"/>
+    <xacro:property name="caster_wheel_mass" value="0.1"/>
     <xacro:property name="caster_wheel_offset_x" value="0.075"/><!---->
     <xacro:property name="caster_wheel_offset_z" value="${wheel_offset_z - wheel_radius + caster_wheel_radius}"/>
@@ -32,14 +32,12 @@
     </material>
     <!-- BASE LINK -->
-    <link name="base_link">
-    </link>
-    <!-- BASE_FOOTPRINT LINK -->
+    <link name="base_link"/>
     <joint name="base_footprint_joint" type="fixed">
         <parent link="base_link"/>
         <child link="base_footprint"/>
         <origin xyz="0 0 0" rpy="0 0 0"/>
+        <axis xyz="0 0 0"/>
     </joint>
-    <link name="base_footprint">
-    </link>
+    <link name="base_footprint"/>
     <!-- CHASSIS LINK -->
     <joint name="chassis_joint" type="fixed">
@@ -89,5 +87,5 @@
             </geometry>
         </collision>
-        <xacro:inertial_box mass="0.03" x="${chassis_length}" y="${chassis_width}" z="${chassis_height}">
+        <xacro:inertial_box mass="0.005" x="${chassis_length}" y="${chassis_width}" z="${chassis_height}">
             <origin xyz="0.025 0 ${(chassis_height/2)-wheel_offset_z}" rpy="0 0 0"/>
         </xacro:inertial_box>

Commit message: adding camera & obstacle world

File: description/robot_core.xacro (robot description, xacro)
@@ -75,7 +75,7 @@
     <link name="chassis_top">
         <visual>
-            <origin xyz="0.025 0 ${(chassis_height/2)-wheel_offset_z}"/>
+            <origin xyz="0.025 0 ${(chassis_height/3)-wheel_offset_z}"/>
             <geometry>
-                <box size="0.05 ${chassis_width} ${chassis_height}"/>
+                <box size="0.05 ${chassis_width} ${chassis_height/3}"/>
             </geometry>
             <material name="white"/>
