Commit message: basic corrections

File: description/gazebo_control.xacro (robot description, xacro)
@@ -6,5 +6,5 @@
             <left_joint>left_wheel_joint</left_joint>
             <right_joint>right_wheel_joint</right_joint>
-            <wheel_separation>0.086</wheel_separation>
+            <wheel_separation>0.096</wheel_separation>
             <wheel_diameter>0.044</wheel_diameter>
             <!-- Limits -->

File: description/robot_core.xacro (robot description, xacro)
@@ -8,10 +8,10 @@
     <xacro:property name="wheel_radius" value="0.022"/><!---->
     <xacro:property name="wheel_thickness" value="0.017"/><!---->
-    <xacro:property name="wheel_mass" value="0.05"/>
+    <xacro:property name="wheel_mass" value="0.3"/>
     <xacro:property name="wheel_offset_x" value="0.016"/><!---->
     <xacro:property name="wheel_offset_y" value="0.048"/><!---->
     <xacro:property name="wheel_offset_z" value="0.005"/><!---->
     <xacro:property name="caster_wheel_radius" value="0.015"/><!---->
-    <xacro:property name="caster_wheel_mass" value="0.01"/>
+    <xacro:property name="caster_wheel_mass" value="0.2"/>
     <xacro:property name="caster_wheel_offset_x" value="0.075"/><!---->
     <xacro:property name="caster_wheel_offset_z" value="${wheel_offset_z - wheel_radius + caster_wheel_radius}"/>
