Commit message: camera initialisation

File: description/robot.urdf.xacro (robot description, xacro)
@@ -4,3 +4,4 @@
     <!-- <xacro:include filename="gazebo_control.xacro" /> -->
     <xacro:include filename="ros2_control.xacro" />
+    <xacro:include filename="camera.xacro" />
 </robot>

File: description/robot_core.xacro (robot description, xacro)
@@ -2,7 +2,7 @@
 <robot xmlns:xacro="http://www.ros.org/wiki/xacro"  >
     <xacro:include filename="inertial_macros.xacro"/>
-    <xacro:property name="chassis_length" value="0.09"/><!---->
-    <xacro:property name="chassis_width" value="0.07"/><!---->
-    <xacro:property name="chassis_height" value="0.04"/><!---->
+    <xacro:property name="chassis_length" value="0.090"/><!---->
+    <xacro:property name="chassis_width" value="0.070"/><!---->
+    <xacro:property name="chassis_height" value="0.040"/><!---->
     <xacro:property name="chassis_mass" value="1.0"/>
     <xacro:property name="wheel_radius" value="0.022"/><!---->
